Commit message: changed starting position of urdf

File: urdf/arm_science_urdf_v2_2025.urdf (robot description, URDF)
Before this commit: robot arm_science_urdf_v2_2025, 6 links, 5 joints
Joints:
- joint Joint_2: origin xyz=0.049213 1.25E-05 0.0747 rpy=-1.57 0 0 -> xyz=0.049213 1.25E-05 0.0747 rpy=0 0 0
